File: kh8833-poweramp/kh8833-poweramp.kicad_pcb (KiCad board)
At the start: 2 copper layers, 245 x 82 mm, 72 parts, among them J10 Conn_01x03, J11 Conn_01x03, J12 Conn_01x03, J7 Conn_01x03, J8 Conn_01x03, J9 Conn_01x06, U1 TDA2050, U2 TDA2050, U3 TDA2050, U4 TDA2050

Commit message: Add speaker prot - v1.0
Parts:
- removed the ? at (113.5, 53.5)
- added C3: 470uF, Capacitor_THT:CP_Radial_D8.0mm_P5.00mm, F.Cu at (40.6, 81.5)
- added C39: 220uF, Capacitor_THT:CP_Radial_D8.0mm_P5.00mm, F.Cu at (65.5, 66.4)
- added C40: 220uF, Capacitor_THT:CP_Radial_D8.0mm_P5.00mm, F.Cu at (54.9, 81.5)
- added C6: 220uF, Capacitor_THT:CP_Radial_D8.0mm_P5.00mm, F.Cu at (59.0, 97.9)
- added D2: D_Bridge_+-AA, Diode_THT:Diode_Bridge_Round_D9.0mm, F.Cu at (34.5, 69.5)
- added D3: 1N4742A, Diode_THT:D_DO-41_SOD81_P10.16mm_Horizontal, F.Cu at (53.6, 93.5)
- added D4: D_Bridge_+-AA, Diode_THT:Diode_Bridge_Round_D9.0mm, F.Cu at (52.0, 66.5)
- added D5: LED, LED_THT:LED_D5.0mm, F.Cu at (87.2, 87.0)
- added D6: 1N4007, Diode_THT:D_DO-41_SOD81_P10.16mm_Horizontal, F.Cu at (104.1, 85.5)
- added J10: Conn_01x02, TerminalBlock_Phoenix:TerminalBlock_Phoenix_MKDS-1,5-2-5.08_1x02_P5.08mm_Horizontal, F.Cu at (31.2, 89.5)
- added J11: Conn_01x02, TerminalBlock_Phoenix:TerminalBlock_Phoenix_MKDS-1,5-2-5.08_1x02_P5.08mm_Horizontal, F.Cu at (31.2, 76.0)
- added K1: HJR1-2C, Relay_THT:Relay_DPDT_Omron_G5V-2, F.Cu at (98.2, 80.9)
- added K2: HJR1-2C, Relay_THT:Relay_DPDT_Omron_G5V-2, F.Cu at (80.7, 80.9)
- added Q1: BC546, Package_TO_SOT_THT:TO-92L_Inline_Wide, F.Cu at (54.5, 74.5)
- added Q2: BC546, Package_TO_SOT_THT:TO-92L_Inline_Wide, F.Cu at (75.0, 84.5)
- added Q3: BC547, Package_TO_SOT_THT:TO-92L_Inline_Wide, F.Cu at (81.0, 84.5)
- added R1: 22, Resistor_THT:R_Axial_DIN0207_L6.3mm_D2.5mm_P10.16mm_Horizontal, F.Cu at (43.4, 98.5)
- added R18: 10k, Resistor_THT:R_Axial_DIN0207_L6.3mm_D2.5mm_P2.54mm_Vertical, F.Cu at (69.6, 80.5)
- added R19: 10k, Resistor_THT:R_Axial_DIN0207_L6.3mm_D2.5mm_P2.54mm_Vertical, F.Cu at (69.6, 75.5)
- added R20: 10k, Resistor_THT:R_Axial_DIN0207_L6.3mm_D2.5mm_P10.16mm_Horizontal, F.Cu at (106.0, 68.1)
- added R21: 10k, Resistor_THT:R_Axial_DIN0207_L6.3mm_D2.5mm_P2.54mm_Vertical, F.Cu at (69.6, 70.5)
- added R22: 10k, Resistor_THT:R_Axial_DIN0207_L6.3mm_D2.5mm_P2.54mm_Vertical, F.Cu at (62.5, 74.5)
- added R23: 10K, Resistor_THT:R_Axial_DIN0207_L6.3mm_D2.5mm_P2.54mm_Vertical, F.Cu at (67.5, 85.5)
- added R24: 39K, Resistor_THT:R_Axial_DIN0207_L6.3mm_D2.5mm_P10.16mm_Horizontal, F.Cu at (55.1, 88.5)
- added R25: 1k, Resistor_THT:R_Axial_DIN0207_L6.3mm_D2.5mm_P2.54mm_Vertical, F.Cu at (96.5, 89.5)
- added REF**: MountingHole_3.2mm_M3, MountingHole:MountingHole_3.2mm_M3, F.Cu at (113.5, 53.5)
- added RV1: 250K, Potentiometer_THT:Potentiometer_Bourns_3296W_Vertical, F.Cu at (60.0, 79.5)
- F2, F3: footprint Fuse:Fuseholder_Littelfuse_100_series_5x20mm -> Fuse:Fuseholder_Littelfuse_445_030_series_5x20mm
- moved J13 122.5 mm to (99.5, 54.2), turned to 180 degrees
- moved J12 56.7 mm to (82.0, 54.2), turned to 180 degrees
- moved J9 51.6 mm to (31.2, 102.9), turned to -90 degrees
- moved F3 42.3 mm to (39.8, 113.0), turned to 0 degrees
- moved F2 35.9 mm to (39.8, 103.0), turned to 0 degrees
- moved D1 32.7 mm to (65.9, 115.6), turned to 90 degrees
- moved C1 13.4 mm to (102.0, 116.5), turned to -90 degrees
- moved C2 13.4 mm to (102.0, 97.0), turned to -90 degrees
- moved C4 13.4 mm to (81.0, 116.5), turned to -90 degrees
- moved C5 13.4 mm to (81.0, 97.0), turned to -90 degrees
- moved J14 5.00 mm to (121.0, 120.0)
- renumbered C8 to C10, C9 to C11, C10 to C12, C11 to C13, C12 to C14, C13 to C15, C14 to C16, C15 to C17, C16 to C18, C17 to C19, C18 to C20, C19 to C21, C20 to C22, C21 to C23, C22 to C24, C23 to C25, C24 to C26, C25 to C27, C26 to C28, C27 to C29, C28 to C30, C29 to C31, C30 to C32, C31 to C33, C32 to C34, C33 to C35, C34 to C36, C35 to C37, C36 to C38, C3 to C4, C4 to C5, C5 to C7, C6 to C8, C7 to C9, J9 to J1, J11 to J12, J12 to J13, J8 to J14, J10 to J2, J7 to J9, R9 to R10, R10 to R11, R11 to R12, R12 to R13, R13 to R14, R14 to R15, R15 to R16, R16 to R17, R1 to R2, R2 to R3, R3 to R4, R4 to R5, R5 to R6, R6 to R7, R7 to R8, R8 to R9
Connections:
- J12 pad 1: /TDA2050Amp0/OUTPUT -> /Protector de Parlantes/Out-1
- J12 pad 3: /TDA2050Amp1/OUTPUT -> /Protector de Parlantes/Out-2
- J13 pad 1: /TDA2050Amp2/OUTPUT -> /Protector de Parlantes/Out-3
- J13 pad 3: /TDA2050Amp3/OUTPUT -> /Protector de Parlantes/Out-4
- R12 pad 2: /TDA2050Amp2/OUTPUT -> /Protector de Parlantes/In-3
- R13 pad 2: /TDA2050Amp2/OUTPUT -> /Protector de Parlantes/In-3
- R16 pad 2: /TDA2050Amp3/OUTPUT -> /Protector de Parlantes/In-4
- R17 pad 2: /TDA2050Amp3/OUTPUT -> /Protector de Parlantes/In-4
- R4 pad 2: /TDA2050Amp0/OUTPUT -> /Protector de Parlantes/In-1
- R5 pad 2: /TDA2050Amp0/OUTPUT -> /Protector de Parlantes/In-1
- R8 pad 2: /TDA2050Amp1/OUTPUT -> /Protector de Parlantes/In-2
- R9 pad 2: /TDA2050Amp1/OUTPUT -> /Protector de Parlantes/In-2
- U1 pad 4: /TDA2050Amp0/OUTPUT -> /Protector de Parlantes/In-1
- U2 pad 4: /TDA2050Amp1/OUTPUT -> /Protector de Parlantes/In-2
- U3 pad 4: /TDA2050Amp2/OUTPUT -> /Protector de Parlantes/In-3
- U4 pad 4: /TDA2050Amp3/OUTPUT -> /Protector de Parlantes/In-4
Routing:
- net /Protector de Parlantes/In-4: track 0.00 -> 193.8 mm
- net /Protector de Parlantes/In-3: track 0.00 -> 124.0 mm
- net /Protector de Parlantes/In-2: track 0.00 -> 109.4 mm
- net +12V: track 0.00 -> 89.1 mm, vias 0 -> 2
- net Net-(C39-Pad1): track 0.00 -> 72.0 mm
- net /Protector de Parlantes/In-1: track 0.00 -> 48.0 mm
- net +24V: track 515.6 -> 469.3 mm, vias 8 -> 6
- net Net-(C40-Pad1): track 0.00 -> 37.0 mm
- net Net-(D2-Pad3): track 0.00 -> 35.5 mm
- net Net-(D2-Pad4): track 0.00 -> 34.2 mm
- net Net-(C3-Pad1): track 0.00 -> 33.2 mm
- net Net-(D5-Pad1): track 0.00 -> 31.8 mm
- net Net-(D4-Pad2): track 0.00 -> 18.9 mm
- net Net-(D4-Pad1): track 0.00 -> 15.7 mm
- net -24V: track 438.0 -> 424.2 mm
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- added copper zone on B.Cu, net /Protector de Parlantes/In-1
- added copper zone on B.Cu, net /Protector de Parlantes/In-2
- added copper zone on B.Cu, net /Protector de Parlantes/In-3
- added copper zone on B.Cu, net /Protector de Parlantes/In-4
- removed copper zone on B.Cu, net /TDA2050Amp0/OUTPUT
- removed copper zone on B.Cu, net /TDA2050Amp1/OUTPUT
- removed copper zone on B.Cu, net /TDA2050Amp2/OUTPUT
- removed copper zone on B.Cu, net /TDA2050Amp3/OUTPUT
